File: pcb/Radio.sch (KiCad schematic (older format))
At the start: 4 parts, among them U301 Radiometrix_MTX2

Commit message: Added BOM
Parts:
- U301: Farnell Value -> (none)
Changed lines of the file:
@@
 EESchema Schematic File Version 2
+LIBS:woodchuck-rescue
 LIBS:power
 LIBS:device
@@
 LIBS:sma
 LIBS:cga0402mlc-12g
+LIBS:agg-kicad
 LIBS:woodchuck-cache
-EELAYER 27 0
+EELAYER 25 0
 EELAYER END
 $Descr A4 11693 8268
@@
 F 3 "http://www.radiometrix.com/files/additional/mtx2.pdf" H 5550 2900 60  0001 C CNN
 F 4 "Value" H 5550 2900 60  0001 C CNN "Digikey"
-F 5 "Value" H 5550 2900 60  0001 C CNN "Farnell"
-F 6 "Value" H 5550 2900 60  0001 C CNN "Fieldname"
+F 5 "Value" H 5550 2900 60  0001 C CNN "Fieldname"
 	1    5550 2900
 	1    0    0    -1
 $EndComp
 $Comp
-L GND #PWR09
+L GND-RESCUE-woodchuck #PWR09
 U 1 1 565CEF3F
 P 5800 2850
@@
 $EndComp
 $Comp
-L GND #PWR010
+L GND-RESCUE-woodchuck #PWR010
 U 1 1 565CEF57
 P 4550 3550
@@
 Quarter wave ant library removed \n(no pins on the antenna components)\nas it kept placing that one instead of \nthis one now (which was used in avionics14)
 $Comp
-L GND #PWR011
+L GND-RESCUE-woodchuck #PWR011
 U 1 1 565D0220
 P 4050 3550
@@
 $EndComp
 $Comp
-L GND #PWR012
+L GND-RESCUE-woodchuck #PWR012
 U 1 1 565D0231
 P 4050 3100
@@
 $EndComp
 $Comp
-L GND #PWR014
+L GND-RESCUE-woodchuck #PWR014
 U 1 1 565D1392
 P 5650 4000
@@
 $EndComp
 $Comp
-L GND #PWR015
+L GND-RESCUE-woodchuck #PWR015
 U 1 1 565D162B
 P 4250 3550
