File: pcb/Radio.sch (KiCad schematic (older format))
At the start: 4 parts, among them U301 Radiometrix_MTX2

Commit message: Tidy up fields to fix bom errors
Parts:
- A301, D301, U301: Digikey Value -> (none); Fieldname Value -> (none)
- C301: value 100n -> 0.1uF; Digikey Value -> (none); Fieldname Value -> (none)
Changed lines of the file:
@@
 F 2 "Woodchuck:MTX2" H 5550 2900 60  0001 C CNN
 F 3 "http://www.radiometrix.com/files/additional/mtx2.pdf" H 5550 2900 60  0001 C CNN
-F 4 "Value" H 5550 2900 60  0001 C CNN "Digikey"
-F 5 "Value" H 5550 2900 60  0001 C CNN "Fieldname"
+F 4 "" H 5550 2900 60  0001 C CNN ""
+F 5 "" H 5550 2900 60  0001 C CNN
 	1    5550 2900
 	1    0    0    -1
@@
 F 2 "Woodchuck:SMA-142-0701-801" H 4200 3625 60  0001 C CNN
 F 3 "" H 4200 3625 60  0000 C CNN
-F 4 "Value" H 3900 3300 60  0001 C CNN "Digikey"
-F 5 "1608592" H 3900 3300 60  0001 C CNN "Farnell"
-F 6 "Value" H 3900 3300 60  0001 C CNN "Fieldname"
+F 4 "1608592" H 3900 3300 60  0001 C CNN "Farnell"
 	1    3900 3300
 	-1   0    0    1
@@
 P 5650 3800
 F 0 "C301" H 5660 3870 50  0000 L CNN
-F 1 "100n" H 5660 3720 50  0000 L CNN
+F 1 "0.1uF" H 5660 3720 50  0000 L CNN
 F 2 "Woodchuck:C0603" H 5650 3800 60  0001 C CNN
 F 3 "" H 5650 3800 60  0000 C CNN
-F 4 "Value" H 5650 3800 60  0001 C CNN "Digikey"
-F 5 "1759037" H 5650 3800 60  0001 C CNN "Farnell"
-F 6 "Value" H 5650 3800 60  0001 C CNN "Fieldname"
+F 4 "1759037" H 5650 3800 60  0001 C CNN "Farnell"
 	1    5650 3800
 	1    0    0    -1
@@
 F 2 "Woodchuck:R0402" H 4250 3300 60  0001 C BNN
 F 3 "" H 4250 3300 60  0000 C CNN
-F 4 "Value" H 4250 3300 60  0001 C CNN "Digikey"
-F 5 "2368169" H 4250 3300 60  0001 C CNN "Farnell"
-F 6 "Value" H 4250 3300 60  0001 C CNN "Fieldname"
+F 4 "2368169" H 4250 3300 60  0001 C CNN "Farnell"
 	1    4250 3300
 	0    1    1    0
