File: pcb/GPS_Ublox.sch (KiCad schematic (older format))
At the start: 4 parts, among them IC201 u-blox_CAM-M8Q

Commit message: Hide footprints on schematic, fix overlaps
Changed lines of the file:
@@
 F 0 "IC201" H 4900 3450 60  0000 C CNN
 F 1 "u-blox_CAM-M8Q" H 5250 1400 60  0000 C CNN
-F 2 "Woodchuck:UBLOX_CAM_M8Q" H 5400 3550 60  0000 C CNN
+F 2 "Woodchuck:UBLOX_CAM_M8Q" H 5400 3550 60  0001 C CNN
 F 3 "https://www2.u-blox.com/images/downloads/Product_Docs/CAM-M8Q_DataSheet_%28UBX-13004081%29.pdf" H 5550 2000 60  0001 C CNN
 	1    5350 2900
@@
 F 0 "R202" V 6400 3000 50  0000 C CNN
 F 1 "220" V 6300 3000 50  0000 C CNN
-F 2 "Woodchuck:0603" V 6230 3000 30  0000 C CNN
+F 2 "Woodchuck:0603" V 6230 3000 30  0001 C CNN
 F 3 "" H 6300 3000 30  0000 C CNN
 F 4 "Value" H 6300 3000 60  0001 C CNN "Digikey"
@@
 F 0 "R201" V 6150 2900 50  0000 C CNN
 F 1 "220" V 6300 2900 50  0000 C CNN
-F 2 "Woodchuck:0603" V 6230 2900 30  0000 C CNN
+F 2 "Woodchuck:0603" V 6230 2900 30  0001 C CNN
 F 3 "" H 6300 2900 30  0000 C CNN
 F 4 "Value" H 6300 2900 60  0001 C CNN "Digikey"

Commit message: Added BOM
Parts:
- C201: symbol C -> C-RESCUE-woodchuck
- R201, R202: symbol R -> R-RESCUE-woodchuck
Changed lines of the file:
@@
 EESchema Schematic File Version 2
+LIBS:woodchuck-rescue
 LIBS:power
 LIBS:device
@@
 LIBS:sma
 LIBS:cga0402mlc-12g
+LIBS:agg-kicad
 LIBS:woodchuck-cache
-EELAYER 27 0
+EELAYER 25 0
 EELAYER END
 $Descr A4 11693 8268
@@
 $EndComp
 $Comp
-L GND #PWR06
+L GND-RESCUE-woodchuck #PWR06
 U 1 1 56AAB217
 P 4550 4300
@@
 -How are we interfacing to the MCU? DSEL may have to be grounded\n-Embedded antenna?
 $Comp
-L C C201
+L C-RESCUE-woodchuck C201
 U 1 1 56ACB00C
 P 4300 2500
+AR Path="/56ACB00C" Ref="C201"  Part="1"
+AR Path="/56574088/56ACB00C" Ref="C201"  Part="1"
 F 0 "C201" H 4325 2600 50  0000 L CNN
 F 1 "100n" H 4325 2400 50  0000 L CNN
@@
 	4050 2500 4050 2650
 $Comp
-L GND #PWR08
+L GND-RESCUE-woodchuck #PWR08
 U 1 1 56ACB0DE
 P 4050 2650
@@
 NoConn ~ 6050 2700
 $Comp
-L R R202
+L R-RESCUE-woodchuck R202
 U 1 1 56ACBA41
 P 6300 3000
@@
 $EndComp
 $Comp
-L R R201
+L R-RESCUE-woodchuck R201
 U 1 1 56ACBA86
 P 6300 2900

Commit message: Tidy up fields to fix bom errors
Parts:
- C201, R201, R202: Digikey Value -> (none); Fieldname Value -> (none)
- IC201: uputronics (none) -> not_listed
Changed lines of the file:
@@
 F 2 "Woodchuck:UBLOX_CAM_M8Q" H 5400 3550 60  0001 C CNN
 F 3 "https://www2.u-blox.com/images/downloads/Product_Docs/CAM-M8Q_DataSheet_%28UBX-13004081%29.pdf" H 5550 2000 60  0001 C CNN
+F 4 "not_listed" H 5350 2900 60  0001 C CNN "uputronics"
 	1    5350 2900
 	1    0    0    -1
@@
 F 2 "Woodchuck:C0603" H 4338 2350 30  0001 C CNN
 F 3 "" H 4300 2500 60  0000 C CNN
-F 4 "Value" H 4300 2500 60  0001 C CNN "Digikey"
-F 5 "9406140" H 4300 2500 60  0001 C CNN "Farnell"
-F 6 "Value" H 4300 2500 60  0001 C CNN "Fieldname"
+F 4 "9406140" H 4300 2500 60  0001 C CNN "Farnell"
 	1    4300 2500
 	0    -1   -1   0
@@
 F 2 "Woodchuck:0603" V 6230 3000 30  0001 C CNN
 F 3 "" H 6300 3000 30  0000 C CNN
-F 4 "Value" H 6300 3000 60  0001 C CNN "Digikey"
-F 5 "1652857" H 6300 3000 60  0001 C CNN "Farnell"
-F 6 "Value" H 6300 3000 60  0001 C CNN "Fieldname"
+F 4 "1652857" H 6300 3000 60  0001 C CNN "Farnell"
 	1    6300 3000
 	0    1    1    0
@@
 F 2 "Woodchuck:0603" V 6230 2900 30  0001 C CNN
 F 3 "" H 6300 2900 30  0000 C CNN
-F 4 "Value" H 6300 2900 60  0001 C CNN "Digikey"
-F 5 "1652857" H 6300 2900 60  0001 C CNN "Farnell"
-F 6 "Value" H 6300 2900 60  0001 C CNN "Fieldname"
+F 4 "1652857" H 6300 2900 60  0001 C CNN "Farnell"
 	1    6300 2900
 	0    1    1    0
