File: pcb/microcontroller.sch (KiCad schematic (older format))
At the start: 24 parts, among them IC1 24AA01, J401 JSTA-4, P401 SWD, P402 USB_OTG, SW401 SPST, U401 STM32F072CBT6, X401 Mounting hole, X402 Mounting hole, X403 CUSF LOGO, X404 CUSF LOGO BACK

Commit message: Added a few missing datasheets and Farnell codes. Still missing GPS and MTX Farnell entry
Parts:
- SW401: Farnell (none) -> 1333652
- U401: Farnell Value -> 2432094
Changed lines of the file:
@@
 F 1 "SPST" H 8550 4650 50  0000 C CNN
 F 2 "Woodchuck:B3U-1000P_switch" H 8550 4950 60  0000 C CNN
-F 3 "" H 8550 4750 60  0000 C CNN
+F 3 "http://www.farnell.com/datasheets/1685550.pdf" H 8550 4750 60  0000 C CNN
+F 4 "1333652" H 8550 4750 60  0001 C CNN "Farnell"
 	1    8550 4750
 	1    0    0    -1
@@
 F 1 "STM32F072CBT6" H 6300 2850 60  0000 C CNN
 F 2 "Woodchuck:LQFP48" H 5400 2900 60  0001 C CNN
-F 3 "" H 5400 2900 60  0000 C CNN
+F 3 "http://www.farnell.com/datasheets/2006534.pdf" H 5400 2900 60  0000 C CNN
 F 4 "Value" H 5050 2800 60  0001 C CNN "Digikey"
-F 5 "Value" H 5050 2800 60  0001 C CNN "Farnell"
+F 5 "2432094" H 5050 2800 60  0001 C CNN "Farnell"
 F 6 "Value" H 5050 2800 60  0001 C CNN "Fieldname"
 	1    5050 2800

Commit message: Hide footprints on schematic, fix overlaps
Connections:
- wire segments 101 -> 121
Other:
- moved on the sheet: D401, R401, R402, R403

Commit message: Fix some layout issues
Connections:
- wire segments 121 -> 100
Changed lines of the file:
@@
 	5800 5400 5800 5500
 Wire Wire Line
-	5800 5500 5900 5500
-Wire Wire Line
-	5900 5500 6000 5500
-Wire Wire Line
-	6000 5500 6100 5500
-Wire Wire Line
-	5900 5400 5900 5500
-Wire Wire Line
-	5900 5500 5900 5600
+	5800 5500 6100 5500
+Wire Wire Line
+	5900 5400 5900 5600
 Connection ~ 5900 5500
 Wire Wire Line
 	6000 5500 6000 5400
 Wire Wire Line
-	5800 2400 5800 2500
-Wire Wire Line
-	5800 2500 5800 2600
+	5800 2400 5800 2600
 Wire Wire Line
 	5700 2600 5700 2500
 Wire Wire Line
-	5600 2500 5700 2500
-Wire Wire Line
-	5700 2500 5800 2500
-Wire Wire Line
-	5800 2500 5900 2500
-Wire Wire Line
-	3000 1650 3000 1750
-Wire Wire Line
-	3000 1750 3000 1850
-Wire Wire Line
-	3000 2150 3000 2250
-Wire Wire Line
-	3000 2250 3000 2350
+	5600 2500 5900 2500
+Wire Wire Line
+	3000 1650 3000 1850
+Wire Wire Line
+	3000 2150 3000 2350
 Connection ~ 3000 2250
 Wire Wire Line
@@
 Connection ~ 3000 1750
 Wire Wire Line
-	2750 2250 3000 2250
-Wire Wire Line
-	3000 2250 3250 2250
-Wire Wire Line
-	3250 2250 3500 2250
-Wire Wire Line
-	2750 1750 3000 1750
-Wire Wire Line
-	3000 1750 3250 1750
-Wire Wire Line
-	3250 1750 3500 1750
-Wire Wire Line
-	1650 1750 1650 1800
-Wire Wire Line
-	1650 1800 1650 1850
+	2750 2250 3500 2250
+Wire Wire Line
+	2750 1750 3500 1750
+Wire Wire Line
+	1650 1750 1650 1850
 Wire Wire Line
 	3250 1750 3250 1850
@@
 	1700 3650 1800 3650
 Wire Wire Line
-	1700 3350 1700 3450
-Wire Wire Line
-	1700 3450 1700 3650
-Wire Wire Line
-	1700 3650 1700 3750
+	1700 3350 1700 3750
 Wire Wire Line
 	1800 3450 1700 3450
@@
 	1800 6550 1800 5550
 Wire Wire Line
-	7850 4750 7950 4750
-Wire Wire Line
-	7950 4750 8050 4750
+	7850 4750 8050 4750
 Wire Wire Line
 	9050 4750 9150 4750
@@
 	9250 5650 9250 4400
 Wire Wire Line
-	1650 2150 1650 2200
-Wire Wire Line
-	1650 2200 1650 2250
+	1650 2150 1650 2250
 Wire Wire Line
 	6700 3350 6900 3350
@@
 	8650 3650 8850 3650
 Wire Wire Line
-	8850 3650 8850 3750
-Wire Wire Line
-	8850 3750 8850 3800
+	8850 3650 8850 3800
 Wire Wire Line
 	8850 3350 8850 3250
@@
 	7600 4200 6700 4200
 Wire Wire Line
-	7600 3350 7600 3500
-Wire Wire Line
-	7600 3500 7600 4200
+	7600 3350 7600 4200
 Wire Wire Line
 	7600 3500 7900 3500
@@
 	7900 3400 7700 3400
 Wire Wire Line
-	7700 3350 7700 3400
-Wire Wire Line
-	7700 3400 7700 4300
+	7700 3350 7700 4300
 Wire Wire Line
 	7700 4300 6700 4300
@@
 	7600 2850 7600 2800
 Wire Wire Line
-	7600 2800 7650 2800
-Wire Wire Line
-	7650 2800 7700 2800
+	7600 2800 7700 2800
 Wire Wire Line
 	7700 2800 7700 2850

Commit message: Added Farnell codes for capacitors
Parts:
- C405: Farnell (none) -> 2496935
- C406: Farnell (none) -> 1535567
Changed lines of the file:
@@
 LIBS:sma
 LIBS:cga0402mlc-12g
-LIBS:agg-kicad
 LIBS:woodchuck-cache
-EELAYER 25 0
+EELAYER 27 0
 EELAYER END
 $Descr A4 11693 8268
@@
 Sheet 4 5
 Title ""
-Date ""
+Date "8 may 2016"
 Rev ""
 Comp ""
@@
 F 2 "Woodchuck:C0603" H 3500 1700 50  0001 C CNN
 F 3 "" H 3500 2000 50  0000 C CNN
+F 4 "1535567" H 3500 2000 60  0001 C CNN "Farnell"
 	1    3500 2000
 	1    0    0    -1
@@
 F 2 "Woodchuck:C0603" H 2050 1750 50  0001 C CNN
 F 3 "" H 2050 2000 50  0000 C CNN
+F 4 "2496935" H 2050 2000 60  0001 C CNN "Farnell"
 	1    2050 2000
 	1    0    0    -1

Commit message: Added BOM
Parts:
- C1, C401, C402, C403, C404, C405, C406: symbol C -> C-RESCUE-woodchuck
- P402: Farnell 2426381 -> 1125348
Changed lines of the file:
@@
 EESchema Schematic File Version 2
+LIBS:woodchuck-rescue
 LIBS:power
 LIBS:device
@@
 LIBS:sma
 LIBS:cga0402mlc-12g
+LIBS:agg-kicad
 LIBS:woodchuck-cache
-EELAYER 27 0
+EELAYER 25 0
 EELAYER END
 $Descr A4 11693 8268
@@
 $EndDescr
 $Comp
-L GND #PWR016
+L GND-RESCUE-woodchuck #PWR016
 U 1 1 565B23CF
 P 5900 5600
@@
 $EndComp
 $Comp
-L C C403
+L C-RESCUE-woodchuck C403
 U 1 1 565B2484
 P 3000 2000
+AR Path="/565B2484" Ref="C403"  Part="1"
+AR Path="/56574098/565B2484" Ref="C403"  Part="1"
 F 0 "C403" H 3025 2100 50  0000 L CNN
 F 1 "0.1uF" H 3025 1900 50  0000 L CNN
@@
 $EndComp
 $Comp
-L GND #PWR017
+L GND-RESCUE-woodchuck #PWR017
 U 1 1 565B2D06
 P 3000 2350
@@
 $EndComp
 $Comp
-L C C402
+L C-RESCUE-woodchuck C402
 U 1 1 565B2D3B
 P 2750 2000
+AR Path="/565B2D3B" Ref="C402"  Part="1"
+AR Path="/56574098/565B2D3B" Ref="C402"  Part="1"
 F 0 "C402" H 2775 2100 50  0000 L CNN
 F 1 "0.1uF" H 2775 1900 50  0000 L CNN
@@
 NOTE: Place one near each\nVDD pin (24, 48) and one\nnear VDDIO2 (36)
 $Comp
-L C C401
+L C-RESCUE-woodchuck C401
 U 1 1 565B339D
 P 1650 2000
+AR Path="/565B339D" Ref="C401"  Part="1"
+AR Path="/56574098/565B339D" Ref="C401"  Part="1"
 F 0 "C401" H 1675 2100 50  0000 L CNN
 F 1 "10nF" H 1675 1900 50  0000 L CNN
@@
 $EndComp
 $Comp
-L GND #PWR018
+L GND-RESCUE-woodchuck #PWR018
 U 1 1 565B33AB
 P 1650 2250
@@
 NOTE: Place near VDDA (9)
 $Comp
-L C C404
+L C-RESCUE-woodchuck C404
 U 1 1 565B3429
 P 3250 2000
+AR Path="/565B3429" Ref="C404"  Part="1"
+AR Path="/56574098/565B3429" Ref="C404"  Part="1"
 F 0 "C404" H 3275 2100 50  0000 L CNN
 F 1 "0.1uF" H 3275 1900 50  0000 L CNN
@@
 SWCLK
 $Comp
-L GND #PWR019
+L GND-RESCUE-woodchuck #PWR019
 U 1 1 565B4620
 P 1700 3750
@@
 EXT_RX
 $Comp
-L GND #PWR020
+L GND-RESCUE-woodchuck #PWR020
 U 1 1 565B6C28
 P 2200 5000
@@
 EXT PORT
 $Comp
-L GND #PWR021
+L GND-RESCUE-woodchuck #PWR021
 U 1 1 565B80EF
 P 2400 6100
@@
 $EndComp
 $Comp
-L GND #PWR022
+L GND-RESCUE-woodchuck #PWR022
 U 1 1 565B8112
 P 2800 6300
@@
 $EndComp
 $Comp
-L GND #PWR023
+L GND-RESCUE-woodchuck #PWR023
 U 1 1 565BAC22
 P 7950 5450
@@
 F 3 "" V 2650 5750 60  0000 C CNN
 F 4 "Value" H 2700 5850 60  0001 C CNN "Digikey"
-F 5 "2426381" H 2700 5850 60  0001 C CNN "Farnell"
+F 5 "1125348" H 2700 5850 60  0001 C CNN "Farnell"
 F 6 "Value" H 2700 5850 60  0001 C CNN "Fieldname"
 	1    2700 5850
@@
 $EndComp
 $Comp
-L C C1
+L C-RESCUE-woodchuck C1
 U 1 1 56BF5C75
 P 8850 3500
+AR Path="/56BF5C75" Ref="C1"  Part="1"
+AR Path="/56574098/56BF5C75" Ref="C1"  Part="1"
 F 0 "C1" H 8875 3600 50  0000 L CNN
 F 1 "0.1uF" H 8875 3400 50  0000 L CNN
@@
 $EndComp
 $Comp
-L GND #PWR030
+L GND-RESCUE-woodchuck #PWR030
 U 1 1 56BF61FD
 P 8850 3800
@@
 NoConn ~ 6700 5100
 $Comp
-L C C406
+L C-RESCUE-woodchuck C406
 U 1 1 56C45ED5
 P 3500 2000
+AR Path="/56C45ED5" Ref="C406"  Part="1"
+AR Path="/56574098/56C45ED5" Ref="C406"  Part="1"
 F 0 "C406" H 3525 2100 50  0000 L CNN
 F 1 "4u7" H 3525 1900 50  0000 L CNN
@@
 $EndComp
 $Comp
-L C C405
+L C-RESCUE-woodchuck C405
 U 1 1 56C46154
 P 2050 2000
+AR Path="/56C46154" Ref="C405"  Part="1"
+AR Path="/56574098/56C46154" Ref="C405"  Part="1"
 F 0 "C405" H 2075 2100 50  0000 L CNN
 F 1 "1u" H 2075 1900 50  0000 L CNN

Commit message: Tidy up fields to fix bom errors
Parts:
- C1, C401, C402, C403, C404, D401, J401, P401, P402, R401, R402, R403, U401: Digikey Value -> (none); Fieldname Value -> (none)
- R1, R2, R404: value 10K -> 10k; Digikey Value -> (none); Fieldname Value -> (none)
Changed lines of the file:
@@
 F 2 "Woodchuck:C0603" H 3050 1800 30  0001 C CNN
 F 3 "" H 3000 2000 60  0000 C CNN
-F 4 "Value" H 3000 2000 60  0001 C CNN "Digikey"
-F 5 "1759037" H 3000 2000 60  0001 C CNN "Farnell"
-F 6 "Value" H 3000 2000 60  0001 C CNN "Fieldname"
+F 4 "1759037" H 3000 2000 60  0001 C CNN "Farnell"
 	1    3000 2000
 	1    0    0    -1
@@
 F 2 "Woodchuck:C0603" H 2788 1850 30  0001 C CNN
 F 3 "" H 2750 2000 60  0000 C CNN
-F 4 "Value" H 2750 2000 60  0001 C CNN "Digikey"
-F 5 "1759037" H 2750 2000 60  0001 C CNN "Farnell"
-F 6 "Value" H 2750 2000 60  0001 C CNN "Fieldname"
+F 4 "1759037" H 2750 2000 60  0001 C CNN "Farnell"
 	1    2750 2000
 	1    0    0    -1
@@
 F 2 "Woodchuck:C0603" H 1688 1850 30  0001 C CNN
 F 3 "" H 1650 2000 60  0000 C CNN
-F 4 "Value" H 1650 2000 60  0001 C CNN "Digikey"
-F 5 "1907314" H 1650 2000 60  0001 C CNN "Farnell"
-F 6 "Value" H 1650 2000 60  0001 C CNN "Fieldname"
+F 4 "1907314" H 1650 2000 60  0001 C CNN "Farnell"
 	1    1650 2000
 	1    0    0    -1
@@
 F 2 "Woodchuck:C0603" H 3288 1850 30  0001 C CNN
 F 3 "" H 3250 2000 60  0000 C CNN
-F 4 "Value" H 3250 2000 60  0001 C CNN "Digikey"
-F 5 "1759037" H 3250 2000 60  0001 C CNN "Farnell"
-F 6 "Value" H 3250 2000 60  0001 C CNN "Fieldname"
+F 4 "1759037" H 3250 2000 60  0001 C CNN "Farnell"
 	1    3250 2000
 	1    0    0    -1
@@
 F 2 "Woodchuck:FTSH-105-01-F-D-K" H 2650 3250 60  0001 C CNN
 F 3 "" H 2650 3250 60  0000 C CNN
-F 4 "Value" H 2300 3450 60  0001 C CNN "Digikey"
-F 5 "1865285" H 2300 3450 60  0001 C CNN "Farnell"
-F 6 "Value" H 2300 3450 60  0001 C CNN "Fieldname"
+F 4 "1865285" H 2300 3450 60  0001 C CNN "Farnell"
 	1    2300 3450
 	1    0    0    -1
@@
 F 2 "Woodchuck:S04B-PASK-2" H 2500 4650 60  0001 C CNN
 F 3 "" H 2500 4650 60  0000 C CNN
-F 4 "Value" H 2500 4550 60  0001 C CNN "Digikey"
-F 5 "1830749" H 2500 4550 60  0001 C CNN "Farnell"
-F 6 "Value" H 2500 4550 60  0001 C CNN "Fieldname"
+F 4 "1830749" H 2500 4550 60  0001 C CNN "Farnell"
 	1    2500 4550
 	1    0    0    -1
@@
 P 7950 5100
 F 0 "R404" H 8070 5190 60  0000 C CNN
-F 1 "10K" H 7950 4950 60  0000 C CNN
+F 1 "10k" H 7950 4950 60  0000 C CNN
 F 2 "Woodchuck:0603" H 7950 4850 60  0001 C CNN
-F 3 "" H 7950 5100 60  0000 C CNN
-F 4 "Value" H 7950 5100 60  0001 C CNN "Digikey"
-F 5 "9331700" H 7950 5100 60  0001 C CNN "Farnell"
-F 6 "Value" H 7950 5100 60  0001 C CNN "Fieldname"
+F 4 "9331700" H 7950 5100 60  0001 C CNN "Farnell"
 	1    7950 5100
 	0    1    1    0
@@
 F 2 "Woodchuck:0603" H 3750 3700 60  0001 C CNN
 F 3 "" H 3750 3700 60  0000 C CNN
-F 4 "Value" H 3750 3700 60  0001 C CNN "Digikey"
-F 5 "1469826" H 3750 3700 60  0001 C CNN "Farnell"
-F 6 "Value" H 3750 3700 60  0001 C CNN "Fieldname"
+F 4 "1469826" H 3750 3700 60  0001 C CNN "Farnell"
 	1    3750 3700
 	1    0    0    -1
@@
 F 2 "Woodchuck:0603" H 4150 4100 60  0001 C CNN
 F 3 "" H 4150 4100 60  0000 C CNN
-F 4 "Value" H 4150 4100 60  0001 C CNN "Digikey"
-F 5 "1469826" H 4150 4100 60  0001 C CNN "Farnell"
-F 6 "Value" H 4150 4100 60  0001 C CNN "Fieldname"
+F 4 "1469826" H 4150 4100 60  0001 C CNN "Farnell"
 	1    4150 4100
 	1    0    0    1
@@
 F 2 "Woodchuck:0603" H 4500 4200 60  0001 C CNN
 F 3 "" H 4500 4200 60  0000 C CNN
-F 4 "Value" H 4500 4200 60  0001 C CNN "Digikey"
-F 5 "1469826" H 4500 4200 60  0001 C CNN "Farnell"
-F 6 "Value" H 4500 4200 60  0001 C CNN "Fieldname"
+F 4 "1469826" H 4500 4200 60  0001 C CNN "Farnell"
 	1    4500 4200
 	1    0    0    -1
@@
 F 2 "Woodchuck:LQFP48" H 5400 2900 60  0001 C CNN
 F 3 "http://www.farnell.com/datasheets/2006534.pdf" H 5400 2900 60  0001 C CNN
-F 4 "Value" H 5050 2800 60  0001 C CNN "Digikey"
-F 5 "2432094" H 5050 2800 60  0001 C CNN "Farnell"
-F 6 "Value" H 5050 2800 60  0001 C CNN "Fieldname"
+F 4 "2432094" H 5050 2800 60  0001 C CNN "Farnell"
 	1    5050 2800
 	1    0    0    -1
@@
 F 2 "Woodchuck:MOLEX_67503_1020_MINI_USB" V 2650 5750 60  0001 C CNN
 F 3 "" V 2650 5750 60  0000 C CNN
-F 4 "Value" H 2700 5850 60  0001 C CNN "Digikey"
-F 5 "1125348" H 2700 5850 60  0001 C CNN "Farnell"
-F 6 "Value" H 2700 5850 60  0001 C CNN "Fieldname"
+F 4 "1125348" H 2700 5850 60  0001 C CNN "Farnell"
 	1    2700 5850
 	0    1    1    0
@@
 F 2 "Woodchuck:C0603" H 8888 3350 30  0001 C CNN
 F 3 "" H 8850 3500 60  0001 C CNN
-F 4 "Value" H 8850 3500 60  0001 C CNN "Digikey"
-F 5 "1759037" H 8850 3500 60  0001 C CNN "Farnell"
-F 6 "Value" H 8850 3500 60  0001 C CNN "Fieldname"
+F 4 "1759037" H 8850 3500 60  0001 C CNN "Farnell"
 	1    8850 3500
 	1    0    0    -1
@@
 P 7700 3100
 F 0 "R2" H 7550 3200 60  0000 C CNN
-F 1 "10K" H 7700 2950 60  0001 C CNN
+F 1 "10k" H 7700 2950 60  0001 C CNN
 F 2 "Woodchuck:0603" H 7700 3100 60  0001 C CNN
 F 3 "" H 7700 3100 60  0000 C CNN
-F 4 "Value" H 7700 3100 60  0001 C CNN "Digikey"
-F 5 "9331700" H 7700 3100 60  0001 C CNN "Farnell"
-F 6 "Value" H 7700 3100 60  0001 C CNN "Fieldname"
+F 4 "9331700" H 7700 3100 60  0001 C CNN "Farnell"
 	1    7700 3100
 	0    1    1    0
@@
 P 7600 3100
 F 0 "R1" H 7450 3000 60  0000 C CNN
-F 1 "10K" H 7600 2950 60  0001 C CNN
+F 1 "10k" H 7600 2950 60  0001 C CNN
 F 2 "Woodchuck:0603" H 7600 3100 60  0001 C CNN
 F 3 "" H 7600 3100 60  0000 C CNN
-F 4 "Value" H 7600 3100 60  0001 C CNN "Digikey"
-F 5 "9331700" H 7600 3100 60  0001 C CNN "Farnell"
-F 6 "Value" H 7600 3100 60  0001 C CNN "Fieldname"
+F 4 "9331700" H 7600 3100 60  0001 C CNN "Farnell"
 	1    7600 3100
 	0    1    1    0
@@
 F 2 "Woodchuck:CREE_RGB_LED" H 3550 5050 50  0001 C CNN
 F 3 "http://www.farnell.com/datasheets/1965387.pdf" H 3500 4950 50  0001 C CNN
-F 4 "Value" H 3600 4550 60  0001 C CNN "Digikey"
-F 5 "2093940" H 3600 4550 60  0001 C CNN "Farnell"
-F 6 "Value" H 3600 4550 60  0001 C CNN "Fieldname"
+F 4 "2093940" H 3600 4550 60  0001 C CNN "Farnell"
 	1    3600 4550
 	0    -1   1    0
