File: woodchuck_2/pcb/woodchuck_2.sch (KiCad schematic (older format))
At the start: 48 parts, among them IC1 Si4460, IC2 24AA01, IC3 ADP3335, IC4 MAX-7Q, P1 SWD, P2 COAX, P3 CONN_01X02, P4 COAX, U1 STM32F072CBT6, X1 Mounting hole, X2 Mounting hole, X3 CUSF LOGO, X4 CUSF LOGO BACK, Y1 TCXO

Commit message: Route Woodchuck 2
Parts:
- removed TP1: TESTPAD, agg:TESTPAD, symbol TESTPAD
- removed X2: Mounting hole, Woodchuck:M3_MOUNT, symbol PART
- X2: renamed from X4; footprint Woodchuck:cusf_logo_full -> Woodchuck:cusf_logo_small; Digikey (none) -> Value; Farnell (none) -> Value; Fieldname (none) -> Value
- X3: value CUSF LOGO -> WOODCHUCK; footprint Woodchuck:cusf_logo -> Woodchuck:Woodchuck_2; Digikey (none) -> Value; Farnell (none) -> Value; Fieldname (none) -> Value
Connections:
- net at R1.1: now also U1.25 (PB12); no longer D1.2 (A)
- net at R1.2: now also D1.2 (A); no longer U1.16 (PA6)
Other:
- moved on the sheet: D1, R1, X2
Changed lines of the file:
@@
 NoConn ~ 6000 3800
 NoConn ~ 6000 3900
-NoConn ~ 6000 4200
 NoConn ~ 4150 4000
 NoConn ~ 4150 3800
@@
 L RESISTOR R1
 U 1 1 56D649F7
-P 3300 3650
-F 0 "R1" H 3150 3700 60  0000 C CNN
-F 1 "510" H 3300 3500 60  0001 C CNN
-F 2 "agg:0402" H 3300 3650 60  0001 C CNN
-F 3 "" H 3300 3650 60  0000 C CNN
-F 4 "Value" H 3300 3650 60  0001 C CNN "Digikey"
-F 5 "2073095" H 3300 3650 60  0001 C CNN "Farnell"
-F 6 "Value" H 3300 3650 60  0001 C CNN "Fieldname"
-	1    3300 3650
+P 6300 4200
+F 0 "R1" H 6150 4250 60  0000 C CNN
+F 1 "510" H 6300 4050 60  0001 C CNN
+F 2 "agg:0402" H 6300 4200 60  0001 C CNN
+F 3 "" H 6300 4200 60  0000 C CNN
+F 4 "Value" H 6300 4200 60  0001 C CNN "Digikey"
+F 5 "2073095" H 6300 4200 60  0001 C CNN "Farnell"
+F 6 "Value" H 6300 4200 60  0001 C CNN "Fieldname"
+	1    6300 4200
 	1    0    0    -1
 $EndComp
@@
 $EndComp
 $Comp
-L PART X2
-U 1 1 56D64AF2
-P 5050 1250
-F 0 "X2" H 5100 1350 50  0000 L CNN
-F 1 "Mounting hole" H 5100 1250 50  0000 L CNN
-F 2 "Woodchuck:M3_MOUNT" H 5050 1250 50  0001 C CNN
-F 3 "" H 5050 1250 50  0001 C CNN
-	1    5050 1250
-	1    0    0    -1
-$EndComp
-$Comp
 L PART X1
 U 1 1 56D64AF9
@@
 $EndComp
 $Comp
-L PART X3
-U 1 1 56D64B00
-P 5800 900
-F 0 "X3" H 5850 1000 50  0000 L CNN
-F 1 "CUSF LOGO" H 5850 900 50  0000 L CNN
-F 2 "Woodchuck:cusf_logo" H 5800 900 50  0001 C CNN
-F 3 "" H 5800 900 50  0001 C CNN
-	1    5800 900
-	1    0    0    -1
-$EndComp
-$Comp
-L PART X4
+L PART X2
 U 1 1 56D64B07
-P 5800 1250
-F 0 "X4" H 5850 1350 50  0000 L CNN
-F 1 "CUSF LOGO BACK" H 5850 1250 50  0000 L CNN
-F 2 "Woodchuck:cusf_logo_full" H 5800 1250 50  0001 C CNN
-F 3 "" H 5800 1250 50  0001 C CNN
-	1    5800 1250
+P 5700 900
+F 0 "X2" H 5750 1000 50  0000 L CNN
+F 1 "CUSF LOGO BACK" H 5750 900 50  0000 L CNN
+F 2 "Woodchuck:cusf_logo_small" H 5700 900 50  0001 C CNN
+F 3 "" H 5700 900 50  0001 C CNN
+F 4 "Value" H 5700 900 60  0001 C CNN "Digikey"
+F 5 "Value" H 5700 900 60  0001 C CNN "Farnell"
+F 6 "Value" H 5700 900 60  0001 C CNN "Fieldname"
+	1    5700 900
 	1    0    0    -1
 $EndComp
@@
 L LED D1
 U 1 1 56E487CC
-P 2950 3950
-F 0 "D1" H 2950 4050 50  0000 C CNN
-F 1 "GRN_LED" H 2950 3850 50  0000 C CNN
-F 2 "agg:0603-LED" H 2950 3950 60  0001 C CNN
-F 3 "" H 2950 3950 60  0000 C CNN
-F 4 "Value" H 2950 3950 60  0001 C CNN "Digikey"
-F 5 "2290328" H 2950 3950 60  0001 C CNN "Farnell"
-F 6 "Value" H 2950 3950 60  0001 C CNN "Fieldname"
-	1    2950 3950
+P 6550 4500
+F 0 "D1" H 6550 4600 50  0000 C CNN
+F 1 "GRN_LED" H 6550 4400 50  0000 C CNN
+F 2 "agg:0603-LED" H 6550 4500 60  0001 C CNN
+F 3 "" H 6550 4500 60  0000 C CNN
+F 4 "Value" H 6550 4500 60  0001 C CNN "Digikey"
+F 5 "2290328" H 6550 4500 60  0001 C CNN "Farnell"
+F 6 "Value" H 6550 4500 60  0001 C CNN "Fieldname"
+	1    6550 4500
 	0    -1   -1   0
 $EndComp
@@
 $EndComp
 $Comp
-L TESTPAD TP1
-U 1 1 56E540B9
-P 6050 2450
-F 0 "TP1" H 6050 2500 50  0000 L CNN
-F 1 "TESTPAD" H 6050 2375 50  0001 L CNN
-F 2 "agg:TESTPAD" H 6050 2300 50  0001 L CNN
-F 3 "" H 6050 2450 50  0001 C CNN
-	1    6050 2450
-	0    -1   -1   0
-$EndComp
-$Comp
 L +3.3V #PWR025
 U 1 1 56E58E19
@@
 Connection ~ 950  1600
 Connection ~ 950  1200
-Wire Wire Line
-	3950 3650 3950 3600
-Wire Wire Line
-	3550 3650 3950 3650
 Connection ~ 6950 2200
 Wire Wire Line
@@
 Wire Wire Line
 	7800 2800 8000 2800
-Wire Wire Line
-	3950 3600 4150 3600
 Connection ~ 5300 4900
 Wire Wire Line
@@
 Wire Wire Line
 	6600 2500 6600 2600
-Wire Wire Line
-	6050 2450 6050 2500
-Connection ~ 6050 2500
 Wire Wire Line
 	750  2450 750  2600
@@
 L GND #PWR031
 U 1 1 56E8878F
-P 2950 4250
-F 0 "#PWR031" H 2950 4000 50  0001 C CNN
-F 1 "GND" H 2950 4100 50  0000 C CNN
-F 2 "" H 2950 4250 60  0000 C CNN
-F 3 "" H 2950 4250 60  0000 C CNN
-	1    2950 4250
-	1    0    0    -1
-$EndComp
-Wire Wire Line
-	2950 3750 2950 3650
-Wire Wire Line
-	2950 3650 3050 3650
-Wire Wire Line
-	2950 4250 2950 4150
+P 6550 4800
+F 0 "#PWR031" H 6550 4550 50  0001 C CNN
+F 1 "GND" H 6550 4650 50  0000 C CNN
+F 2 "" H 6550 4800 60  0000 C CNN
+F 3 "" H 6550 4800 60  0000 C CNN
+	1    6550 4800
+	1    0    0    -1
+$EndComp
+Wire Wire Line
+	6550 4800 6550 4700
 $Comp
 L C C21
@@
 Wire Wire Line
 	1800 6850 1850 6850
+NoConn ~ 4150 3600
+Wire Wire Line
+	6550 4300 6550 4200
+Wire Wire Line
+	6050 4200 6000 4200
+$Comp
+L PART X3
+U 1 1 56EBA373
+P 5050 1200
+F 0 "X3" H 5100 1300 50  0000 L CNN
+F 1 "WOODCHUCK" H 5100 1200 50  0000 L CNN
+F 2 "Woodchuck:Woodchuck_2" H 5050 1200 50  0001 C CNN
+F 3 "" H 5050 1200 50  0001 C CNN
+F 4 "Value" H 5050 1200 60  0001 C CNN "Digikey"
+F 5 "Value" H 5050 1200 60  0001 C CNN "Farnell"
+F 6 "Value" H 5050 1200 60  0001 C CNN "Fieldname"
+	1    5050 1200
+	1    0    0    -1
+$EndComp
 $EndSCHEMATC
